File: src/MinBoard.kicad_pcb (KiCad board)
At the start: 2 copper layers, 61.2 x 61.9 mm, 19 parts, among them U1 MCU_Seeed_XIAO_RP2040

Commit message: Updated kicad files
Other:
- board size 61.2 x 61.9 mm -> 61.9 x 61.9 mm
Changed lines of the file:
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@@
 			(drillshape 0)
 			(scaleselection 1)
-			(outputdirectory "gerber")
+			(outputdirectory "../gerber/")
 		)
 	)
@@
 		(model "${SCOTTOKEEBS_KICAD}/3dmodels/ScottoKeebs_MCU.3dshapes/Seeed_XIAO_RP2040.step"
 			(offset
-				(xyz 0 0 0)
+				(xyz 0 0 2)
 			)
 			(scale
@@
 			)
 			(rotate
-				(xyz 0 0 0)
+				(xyz -0 -0 -0)
 			)
 		)
@@
 		)
 	)
+	(gr_circle
+		(center 76.17929 59.47929)
+		(end 77.64957 60.94957)
+		(stroke
+			(width 0.05)
+			(type default)
+		)
+		(fill no)
+		(layer "Edge.Cuts")
+	)
+	(gr_circle
+		(center 133.38225 59.47929)
+		(end 134.85253 60.94957)
+		(stroke
+			(width 0.05)
+			(type default)
+		)
+		(fill no)
+		(layer "Edge.Cuts")
+	)
+	(gr_circle
+		(center 133.38225 116.7)
+		(end 134.85253 118.17028)
+		(stroke
+			(width 0.05)
+			(type default)
+		)
+		(fill no)
+		(layer "Edge.Cuts")
+	)
+	(gr_circle
+		(center 76.2 116.7)
+		(end 77.67028 118.17028)
+		(stroke
+			(width 0.05)
+			(type default)
+		)
+		(fill no)
+		(layer "Edge.Cuts")
+	)
 	(gr_rect
 		(start 73.81875 57.15)
-		(end 135.0645 119.0625)
+		(end 135.7645 119.0625)
 		(stroke
 			(width 0.05)
